Commit message: save

File: assets/urdf/UsefulHound/urdf/Hound.urdf (robot description, URDF)
Before this commit: robot Hound_description, 24 links, 23 joints
Joints:
- joint fixed: origin (none) -> xyz=0.15 0 0.05 rpy=0 0 0

Commit message: mani_exp1_osc_vs_joint

File: assets/urdf/UsefulHound/urdf/Hound.urdf (robot description, URDF)
Before this commit: robot UsefulHound, 24 links, 23 joints
Joints:
- joint fixed: origin xyz=0.15 0 0.05 rpy=0 0 0 -> xyz=0 0 0 rpy=0 0 0
